File: Modules/Controller/Babys_First_Control_Card/first_ctrl_card/first_ctrl_card.kicad_pcb (KiCad board)
At the start: 4 copper layers, 95 x 72.5 mm, 46 parts, among them J1 Clean_Card_v1, J2 RJ45_Shielded, J3 Micro_SD_Card_Det1, J4 RJ45_Shielded, U1 STM32F446RETx, U2 TCAN337, U3 AP7375-33SA-7, X1 ECS-TXO-2520MV-120-AN-TR, Y1 SC32S-7PF20PPM

Commit message: Woo
Parts:
- removed the R9 at (59.5, 146.3)
- removed the R9 at (30.7, 136.1)
- added C20: 1u, Capacitor_SMD:C_0805_2012Metric, F.Cu at (105.4, 124.3)
- added C21: 1u, Capacitor_SMD:C_0805_2012Metric, B.Cu at (134.5, 96.3)
- added C22: 1u, Capacitor_SMD:C_0805_2012Metric, B.Cu at (134.5, 104.9)
- added C23: 100n, Capacitor_SMD:C_0805_2012Metric, F.Cu at (151.6, 111.4)
- added C24: 100n, Capacitor_SMD:C_0805_2012Metric, F.Cu at (137.8, 108.2)
- added C25: 100n, Capacitor_SMD:C_0805_2012Metric, F.Cu at (154.3, 99.7)
- added C26: 100n, Capacitor_SMD:C_0805_2012Metric, F.Cu at (137.7, 100.9)
- added C27: 1u, Capacitor_SMD:C_0805_2012Metric, F.Cu at (155.1, 97.0)
- added C28: 1u, Capacitor_SMD:C_0805_2012Metric, F.Cu at (137.8, 110.2)
- added C29: 1u, Capacitor_SMD:C_0805_2012Metric, F.Cu at (151.6, 113.4)
- added D1: D_Schottky, Diode_SMD:D_SOD-123, B.Cu at (112.0, 125.5)
- added D10: 5V_PRESENT_LED, LED_SMD:LED_0805_2012Metric, F.Cu at (133.9, 66.0)
- added D11: 5VD_PRESENT_LED, LED_SMD:LED_0805_2012Metric, F.Cu at (126.0, 66.0)
- added D12: BUS_PRESENT_LED, LED_SMD:LED_0805_2012Metric, F.Cu at (110.0, 66.0)
- added D13: 3V_PRESENT_LED, LED_SMD:LED_0805_2012Metric, F.Cu at (149.9, 66.0)
- added D2: D_Schottky, Diode_SMD:D_SOD-123, B.Cu at (116.8, 125.5)
- added D3: D_Zener, Diode_SMD:D_SOD-123, B.Cu at (136.8, 97.5)
- added D4: D_Zener, Diode_SMD:D_SOD-123, B.Cu at (136.8, 103.8)
- added D5: BOOTLED_G, LED_SMD:LED_0805_2012Metric, F.Cu at (157.9, 66.0)
- added D6: BUSPWR_GOOD_G, LED_SMD:LED_0805_2012Metric, F.Cu at (117.9, 66.0)
- added D7: 5V_GOOD_G, LED_SMD:LED_0805_2012Metric, F.Cu at (141.9, 66.0)
- added D8: D_Schottky, Diode_SMD:D_SOD-123, B.Cu at (114.4, 125.5)
- added D9: PROBLEM_LED_R, LED_SMD:LED_0805_2012Metric, F.Cu at (182.0, 66.0)
- added G***: LOGO, LOGO, F.Cu at (158.6, 81.6)
- added P1: USB_C_Plug_USB2.0, Connector_USB:USB_C_Receptacle_GCT_USB4105-xx-A_16P_TopMnt_Horizontal, F.Cu at (95.9, 120.5)
- added Q1: BSS83P, Package_TO_SOT_SMD:SOT-23, F.Cu at (108.2, 124.5)
- added R17: 56k, Resistor_SMD:R_0805_2012Metric, F.Cu at (102.6, 122.3)
- added R18: 56k, Resistor_SMD:R_0805_2012Metric, F.Cu at (102.2, 117.4)
- added R19: 100k, Resistor_SMD:R_0805_2012Metric, F.Cu at (108.1, 119.0)
- added R20: DNI, Resistor_SMD:R_0805_2012Metric, F.Cu at (108.2, 121.4)
- added R21: 220R, Resistor_SMD:R_0805_2012Metric, F.Cu at (182.1, 71.0)
- added R22: 470R, Resistor_SMD:R_0805_2012Metric, F.Cu at (133.9, 71.0)
- added R23: 470R, Resistor_SMD:R_0805_2012Metric, F.Cu at (126.0, 71.0)
- added R24: 3k3, Resistor_SMD:R_0805_2012Metric, F.Cu at (110.0, 71.0)
- added R25: 330R, Resistor_SMD:R_0805_2012Metric, F.Cu at (149.9, 71.0)
- added R26: 4k7, Resistor_SMD:R_0805_2012Metric, B.Cu at (133.5, 111.0)
- added R27: 4k7, Resistor_SMD:R_0805_2012Metric, B.Cu at (131.5, 112.0)
- added R28: 10k, Resistor_SMD:R_0805_2012Metric, B.Cu at (133.8, 99.1)
- added R29: 10k, Resistor_SMD:R_0805_2012Metric, B.Cu at (133.8, 102.1)
- added R9: 100k, Resistor_SMD:R_0805_2012Metric, B.Cu at (130.6, 95.6)
- C1, C10, C12, C13, C14, C15, C16, C17, C18, C2, C9: footprint Capacitor_SMD:C_0603_1608Metric -> Capacitor_SMD:C_0805_2012Metric; moved to B.Cu
- C11, C19, C3, C4, C5, C6, C7, C8: footprint Capacitor_SMD:C_0603_1608Metric -> Capacitor_SMD:C_0805_2012Metric
- FB1, U3: moved to B.Cu
- R1, R14, R15, R16, R2, R3, R4, R5, R6, R7: footprint Resistor_SMD:R_0603_1608Metric -> Resistor_SMD:R_0805_2012Metric
- R10, R11, R12, R13, R8: footprint Resistor_SMD:R_0603_1608Metric -> Resistor_SMD:R_0805_2012Metric; moved to B.Cu
- moved C19 151.1 mm to (168.5, 71.5), turned to 180 degrees
- moved R14 138.2 mm to (157.9, 71.0), turned to 180 degrees
- moved C11 135.8 mm to (168.5, 74.0), turned to 180 degrees
- moved R16 126.7 mm to (141.9, 71.0), turned to 180 degrees
- moved C5 121.6 mm to (143.9, 87.1), turned to 90 degrees
- moved C4 119.8 mm to (152.0, 96.3), turned to 90 degrees
- moved C8 117.0 mm to (150.0, 90.9), turned to 90 degrees
- moved R8 116.9 mm to (153.2, 91.1)
- moved R3 114.9 mm to (141.9, 87.1), turned to -90 degrees
- moved R1 114.8 mm to (158.3, 99.7), turned to 90 degrees
- moved R2 114.7 mm to (156.3, 99.7), turned to -90 degrees
- moved C7 113.6 mm to (147.6, 90.9), turned to 90 degrees
- moved C6 113.2 mm to (145.9, 87.1), turned to 90 degrees
- moved C2 112.0 mm to (145.4, 95.5)
- moved C1 111.6 mm to (145.2, 93.4)
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Connections:
- net /ADC_BATT renamed Net-(R11-Pad2)
- J1 pad B12: /CANH_0 -> /CANL_0
- J1 pad B13: /CANL_0 -> /CANH_0
- R10 pad 1: /ADC_5V -> Net-(R10-Pad1)
- R6 pad 2: Net-(U2-FAULT) -> /CAN_FAULT
- U1 pad 10: unconnected-(U1-PC2-Pad10) -> /ADC_123_IN12
- U1 pad 11: unconnected-(U1-PC3-Pad11) -> /ADC_123_IN13
- U1 pad 14: /ESC_7 -> /ESC_4
- U1 pad 15: /ESC_6 -> /ESC_5
- U1 pad 16: /ESC_5 -> /ESC_6
- U1 pad 17: /ESC_4 -> /ESC_7
- U1 pad 22: /ESC_3 -> /ESC_0
- U1 pad 23: /ESC_2 -> /ESC_1
- U1 pad 26: /ESC_1 -> /ESC_2
- U1 pad 27: /ESC_0 -> /ESC_3
- U1 pad 33: unconnected-(U1-PB12-Pad33) -> /PROBLEM_LED
- U1 pad 34: unconnected-(U1-PB13-Pad34) -> /BOOT_LED
- U1 pad 35: unconnected-(U1-PB14-Pad35) -> /5V_BUS_GOOD_LED
- U1 pad 36: unconnected-(U1-PB15-Pad36) -> /BUS_POWER_GOOD_LED
- U1 pad 44: unconnected-(U1-PA11-Pad44) -> /USB_D-
- U1 pad 45: unconnected-(U1-PA12-Pad45) -> /USB_D+
- U1 pad 56: unconnected-(U1-PB4-Pad56) -> /CAN_FAULT
- U1 pad 8: unconnected-(U1-PC0-Pad8) -> /ADC_123_IN10
- U1 pad 9: unconnected-(U1-PC1-Pad9) -> /ADC_123_IN11
- U2 pad 5: Net-(U2-FAULT) -> /CAN_FAULT
Routing:
- net GND: track 0.00 -> 177.4 mm, vias 0 -> 169
- net +5V: track 0.00 -> 164.7 mm, vias 0 -> 4
- net VBUS: track 0.00 -> 118.7 mm, vias 0 -> 2
- net /PROBLEM_LED: track 0.00 -> 114.8 mm
- net /BOOT_LED: track 0.00 -> 96.0 mm
- net /5V_BUS_GOOD_LED: track 0.00 -> 82.8 mm
- net +5VD: track 0.00 -> 77.8 mm, vias 0 -> 2
- net /BUS_POWER_GOOD_LED: track 0.00 -> 74.8 mm
- net /i2C_SCL: track 0.00 -> 67.5 mm, vias 0 -> 3
- net /i2C_SDA: track 0.00 -> 67.4 mm, vias 0 -> 3
- net /USB_D+: track 0.00 -> 58.5 mm
- net /USB_D-: track 0.00 -> 57.7 mm
- net /CAN_FAULT: track 0.00 -> 46.6 mm, vias 0 -> 2
- net +3V3: track 0.00 -> 45.2 mm, vias 0 -> 17
- net /SD_DAT0: track 0.00 -> 43.9 mm, vias 0 -> 1
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- added copper zone on B.Cu, net +3V3
- added copper zone on In2.Cu, net +3V3
- added copper zone on B.Cu, net GND
- added copper zone on F.Cu, net GND
- added copper zone on In1.Cu, net GND
- added copper zone on In2.Cu, net GND
- added copper zone on B.Cu, net Net-(D1-K)
Other:
- board text added: "3V3 CARD PRESENT"
- board text added: "4S BUS P GOOD"
- board text added: "4S BUS PRESENT"
- board text added: "5V CARD P GOOD"
- board text added: "BUS 5V PRESENT"
- board text added: "CARD BOOT"
- board text added: "CARD PROBLEM!"
- board text added: "Main Control Card v.1 w/ ESC Output Joseph A. De Vico 05/16/2024"
- board text added: "USB 5V PRESENT"
