File: Modules/Controller/Babys_First_Control_Card/first_ctrl_card/first_ctrl_card.kicad_sch (KiCad schematic)
At the start: 1 part, among them J1 Clean_Card_v1

Commit message: Almost done with card profile
Parts:
- added U1: STM32F446RETx, Package_QFP:LQFP-64_10x10mm_P0.5mm, symbol MCU_ST_STM32F4:STM32F446RETx
Connections:
- new net: U1.18 (VSS), U1.31 (VSS), U1.47 (VSS), U1.63 (VSS)
Changed lines of the file:
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@@
 (kicad_sch (version 20230121) (generator eeschema)
   (paper "A4")
-  (symbol (lib_id "10061913-102CLF:Clean_Card_v1") (at 66.04 117.475 0) (unit 1)
+  (symbol (lib_id "10061913-102CLF:Clean_Card_v1") (at 46.355 106.68 0) (unit 1)
     (in_bom yes) (on_board yes) (dnp no) (fields_autoplaced)
-    (property "Reference" "J1" (at 66.04 49.53 0)
+    (property "Reference" "J1" (at 46.355 38.1 0)
       (effects (font (size 1.27 1.27)))
     )
-    (property "Value" "Clean_Card_v1" (at 66.04 52.07 0)
+    (property "Value" "Clean_Card_v1" (at 46.355 40.64 0)
       (effects (font (size 1.27 1.27)))
     )
-    (property "Footprint" "goldmansachs:official_mechatronics_card" (at 66.04 117.475 0)
+    (property "Footprint" "goldmansachs:official_mechatronics_card" (at 46.355 106.68 0)
       (effects (font (size 1.27 1.27)) (justify bottom) hide)
     )
-    (property "Datasheet" "invest in seeds" (at 66.04 117.475 0)
+    (property "Datasheet" "invest in seeds" (at 46.355 106.68 0)
       (effects (font (size 1.27 1.27)) hide)
     )
-    (property "PARTREV" "S" (at 66.04 117.475 0)
+    (property "PARTREV" "S" (at 46.355 106.68 0)
       (effects (font (size 1.27 1.27)) (justify bottom) hide)
     )
-    (property "STANDARD" "Manufacturer Recommendations" (at 66.04 117.475 0)
+    (property "STANDARD" "Manufacturer Recommendations" (at 46.355 106.68 0)
       (effects (font (size 1.27 1.27)) (justify bottom) hide)
     )
-    (property "MAXIMUM_PACKAGE_HEIGHT" "11.10mm" (at 66.04 117.475 0)
+    (property "MAXIMUM_PACKAGE_HEIGHT" "11.10mm" (at 46.355 106.68 0)
       (effects (font (size 1.27 1.27)) (justify bottom) hide)
     )
-    (property "MANUFACTURER" "Amphenol" (at 66.04 117.475 0)
+    (property "MANUFACTURER" "Amphenol" (at 46.355 106.68 0)
       (effects (font (size 1.27 1.27)) (justify bottom) hide)
     )
@@
         )
       )
+    )
+  )
+  (symbol (lib_id "MCU_ST_STM32F4:STM32F446RETx") (at 189.865 93.345 0) (unit 1)
+    (in_bom yes) (on_board yes) (dnp no) (fields_autoplaced)
+    (property "Reference" "U1" (at 194.5991 138.43 0)
+      (effects (font (size 1.27 1.27)) (justify left))
+    )
+    (property "Value" "STM32F446RETx" (at 194.5991 140.97 0)
+      (effects (font (size 1.27 1.27)) (justify left))
+    )
+    (property "Footprint" "Package_QFP:LQFP-64_10x10mm_P0.5mm" (at 174.625 136.525 0)
+      (effects (font (size 1.27 1.27)) (justify right) hide)
+    )
+    (property "Datasheet" "https://www.st.com/resource/en/datasheet/stm32f446re.pdf" (at 189.865 93.345 0)
+      (effects (font (size 1.27 1.27)) hide)
+    )
+    (pin "1")
+    (pin "10")
+    (pin "11")
+    (pin "12")
+    (pin "13")
+    (pin "14")
+    (pin "15")
+    (pin "16")
+    (pin "17")
+    (pin "18")
+    (pin "19")
+    (pin "2")
+    (pin "20")
+    (pin "21")
+    (pin "22")
+    (pin "23")
+    (pin "24")
+    (pin "25")
+    (pin "26")
+    (pin "27")
+    (pin "28")
+    (pin "29")
+    (pin "3")
+    (pin "30")
+    (pin "31")
+    (pin "32")
+    (pin "33")
+    (pin "34")
+    (pin "35")
+    (pin "36")
+    (pin "37")
+    (pin "38")
+    (pin "39")
+    (pin "4")
+    (pin "40")
+    (pin "41")
+    (pin "42")
+    (pin "43")
+    (pin "44")
+    (pin "45")
+    (pin "46")
+    (pin "47")
+    (pin "48")
+    (pin "49")
+    (pin "5")
+    (pin "50")
+    (pin "51")
+    (pin "52")
+    (pin "53")
+    (pin "54")
+    (pin "55")
+    (pin "56")
+    (pin "57")
+    (pin "58")
+    (pin "59")
+    (pin "6")
+    (pin "60")
+    (pin "61")
+    (pin "62")
+    (pin "63")
+    (pin "64")
+    (pin "7")
+    (pin "8")
+    (pin "9")
+    (instances
+      (project "first_ctrl_card"
+        (path "/d708b1f2-31af-4742-b27f-f6cfc745df66"
+          (reference "U1") (unit 1)
+        )
+      )

Commit message: Control card dump
Parts:
- added C1, C14, C15, C18: 10u, Capacitor_SMD:C_0603_1608Metric, symbol Device:C_Small
- added C10, C13, C16, C19, C20: 1u, Capacitor_SMD:C_0603_1608Metric, symbol Device:C_Small
- added C11, C12, C17, C2, C4, C5, C9: 100n, Capacitor_SMD:C_0603_1608Metric, symbol Device:C_Small
- added C3: 2u2, Capacitor_SMD:C_0603_1608Metric, symbol Device:C_Small
- added C6: 10n, Capacitor_SMD:C_0603_1608Metric, symbol Device:C_Small
- added C7, C8: 6p, Capacitor_SMD:C_0603_1608Metric, symbol Device:C_Small
- added D1, D2, D8: D_Schottky, symbol Device:D_Schottky
- added D10: 5V_PRESENT_LED, symbol Device:LED
- added D11: 5VD_PRESENT_LED, symbol Device:LED
- added D12: BUS_PRESENT_LED, symbol Device:LED
- added D13: 3V_PRESENT_LED, symbol Device:LED
- added D3, D4: D_Zener, symbol Device:D_Zener
- added D5: BOOTLED_G, symbol Device:LED
- added D6: BUSPWR_GOOD_G, symbol Device:LED
- added D7: 5V_GOOD_G, symbol Device:LED
- added D9: PROBLEM_LED_R, symbol Device:LED
- added FB1: FerriteBead_Small, Inductor_SMD:L_0603_1608Metric, symbol Device:FerriteBead_Small
- added J2, J4: RJ45_Shielded, Connector_RJ:RJ45_Ninigi_GE, symbol Connector:RJ45_Shielded
- added J3: Micro_SD_Card_Det1, goldmansachs:MSD-1-A_SD_CARD_W_DET, symbol Connector:Micro_SD_Card_Det1
- added P1: USB_C_Plug_USB2.0, symbol Connector:USB_C_Plug_USB2.0
- added Q1: BSS83P, Package_TO_SOT_SMD:SOT-23, symbol Transistor_FET:BSS83P
- added R1, R4, R5: 0R, Resistor_SMD:R_0603_1608Metric, symbol Device:R_Small_US
- added R10, R11, R12, R19, R8, R9: 100k, Resistor_SMD:R_0603_1608Metric, symbol Device:R_Small_US
- added R13, R7: 10k, Resistor_SMD:R_0603_1608Metric, symbol Device:R_Small_US
- added R14, R15, R16, R21: 220R, Resistor_SMD:R_0603_1608Metric, symbol Device:R_Small_US
- added R17, R18: 56k, Resistor_SMD:R_0603_1608Metric, symbol Device:R_Small_US
- added R2, R20, R3: DNI, Resistor_SMD:R_0603_1608Metric, symbol Device:R_Small_US
- added R22, R23: 470R, Resistor_SMD:R_0603_1608Metric, symbol Device:R_Small_US
- added R24: 3k3, Resistor_SMD:R_0603_1608Metric, symbol Device:R_Small_US
- added R25: 330R, Resistor_SMD:R_0603_1608Metric, symbol Device:R_Small_US
- added R6: 4k7, Resistor_SMD:R_0603_1608Metric, symbol Device:R_Small_US
- added U2: TCAN337, Package_TO_SOT_SMD:TSOT-23-8, symbol Interface_CAN_LIN:TCAN337
- added U3: AP7375-33SA-7, Package_TO_SOT_SMD:SOT-23-3, symbol ICDB_Waffle:AP7375-33SA-7
- added X1: ECS-TXO-2520MV-120-AN-TR, Oscillator:Oscillator_SMD_ECS_2520MV-xxx-xx-4Pin_2.5x2.0mm, symbol Oscillator:ECS-2520MV-xxx-xx
- added Y1: SC32S-7PF20PPM, MECH_CHIPS:SC32S-7PF20PPM, symbol Device:Crystal
Connections:
- net GND: now reaches J1.B1 (GND), J1.B10 (GND), J1.B11 (GND), J1.B14 (GND), J1.B15 (GND), J1.B20 (GND), J1.B21 (GND), J1.B34 (GND), J1.B35 (GND), J1.B38 (GND), J1.B39 (GND), J1.B44 (GND), J1.B49 (GND), J1.B6 (GND), J1.B7 (GND)
- net GND: now also U1.12 (VSSA), U1.18 (VSS), U1.31 (VSS), U1.47 (VSS), U1.63 (VSS), C1.2, C10.2, C11.2, C12.2, C13.2, C14.2, C15.2, C16.2, C17.2, C18.2, C19.2, C2.2, C20.2, C3.2, C4.2, C5.2, C6.2, C7.2, C8.2, C9.2, D3.2 (A), D4.2 (A), J2.1, J2.3, J2.5, J2.7, J2.SH, J3.10 (SHIELD), J3.6 (VSS), J4.1, J4.3, J4.5, J4.7, J4.SH, P1.A1 (GND), P1.A12 (GND), P1.B1 (GND), P1.B12 (GND), P1.S1 (SHIELD), R1.2, R10.2, R13.2, R14.2, R15.2, R16.2, R17.2, R18.2, R19.2, R21.2, R22.2, R23.2, R24.2, R25.2, R4.2, R7.2, U2.2 (GND), U3.3 (GND), X1.2 (GND)
- net CANH_0: now reaches J1.B12 (CANH_0)
- net CANH_0: now also R5.1, U2.7 (CANH)
- net CANL_0: now reaches J1.B13 (CANL_0)
- net CANL_0: now also R5.2, U2.6 (CANL)
- net +5V: now reaches J1.B16 (5V)
- net +5V: now also J1.B17 (5V), J1.B18 (5V), J1.B19 (5V), D10.2 (A), D2.2 (A), Q1.1 (G), R19.1, R20.2, R9.1
- net VBUS: now reaches J1.B2 (VBATSW)
- net VBUS: now also J1.B3 (VBATSW), J1.B4 (VBATSW), J1.B5 (VBATSW), D1.2 (A), D12.2 (A), R11.1, R12.1
- net DEBUG_UART_RX: now reaches J1.B36 (UART_RX_0)
- net DEBUG_UART_TX: now reaches J1.B37 (UART_TX_0)
- net i2C_SCL: now reaches J1.B8 (I2C_SCL_0)
- net i2C_SCL: now also U1.58 (PB6)
- net i2C_SDA: now reaches J1.B9 (I2C_SDA_0)
- net i2C_SDA: now also U1.59 (PB7)
- net at U1.13 (VDDA): now also C1.1, C2.1, FB1.1
- net ESC_7: now reaches U1.14 (PA0)
- net ESC_7: now also J2.8
- net ESC_6: now reaches U1.15 (PA1)
- net ESC_6: now also J2.6
- net ESC_5: now reaches U1.16 (PA2)
- net ESC_5: now also J2.4
- net ESC_4: now reaches U1.17 (PA3)
- net ESC_4: now also J2.2
- net +3V3: now reaches U1.19 (VDD)
- net +3V3: now also U1.32 (VDD), U1.48 (VDD), U1.64 (VDD), C10.1, C11.1, C15.1, C16.1, C17.1, C18.1, C19.1, C5.1, C6.1, C9.1, D13.2 (A), FB1.2, J3.4 (VDD), R2.1, R3.1, R6.1, R8.1, U2.3 (VCC), U3.2 (VOUT), X1.4 (VDD)
- net ESC_3: now reaches U1.22 (PA6)
- net ESC_3: now also J4.8
- net ESC_2: now reaches U1.23 (PA7)
- net ESC_2: now also J4.6
- net ESC_1: now reaches U1.26 (PB0)
- net ESC_1: now also J4.4
- net ESC_0: now reaches U1.27 (PB1)
- net ESC_0: now also J4.2
- net LSE_I: now reaches U1.3 (PC14)
- net LSE_I: now also C8.1, Y1.2
- net at U1.30 (VCAP_1): now also C3.1
- net SD_DET: now reaches U1.38 (PC7)
- net SD_DET: now also J3.9 (DET), R8.2
- net SD_DAT0: now reaches U1.39 (PC8)
- net SD_DAT0: now also J3.7 (DAT0)
- net LSE_O: now reaches U1.4 (PC15)
- net LSE_O: now also C7.1, Y1.1
- net SD_DAT1: now reaches U1.40 (PC9)
- net SD_DAT1: now also J3.8 (DAT1)
- net USB_DM: now reaches U1.44 (PA11)
- net USB_DP: now reaches U1.45 (PA12)
- net 12MHz_OSC: now reaches U1.5 (PH0)
- net 12MHz_OSC: now also X1.3 (OUT)
- net SD_DAT2: now reaches U1.51 (PC10)
- net SD_DAT2: now also J3.1 (DAT2)
- net SD_DAT3/CD: now reaches U1.52 (PC11)
- net SD_DAT3/CD: now also J3.2 (DAT3/CD)
- net SD_CLK: now reaches U1.53 (PC12)
- net SD_CLK: now also J3.5 (CLK)
- net SD_CMD: now reaches U1.54 (PD2)
- net SD_CMD: now also J3.3 (CMD)
- net CAN_SILENT: now reaches U1.57 (PB5)
- net CAN_SILENT: now also R7.1, U2.8 (S)
- net BOOTLOADER_ENTRY: now reaches U1.60 (BOOT0)
- net BOOTLOADER_ENTRY: now also R1.1, R2.2
- net CAN_RX_0: now reaches U1.61 (PB8)
- net CAN_RX_0: now also U2.4 (RXD)
- net CAN_TX_0: now reaches U1.62 (PB9)
- net CAN_TX_0: now also U2.1 (TXD)
- net ~{RESET}: now reaches U1.7 (NRST)
- net ~{RESET}: now also C4.1
- new net: D7.1 (K), R16.1
- new net: C12.1, C13.1, C14.1, D1.1 (K), D2.1 (K), D8.1 (K), U3.1 (VIN)
- new net: C20.1, P1.A4 (VBUS), P1.A9 (VBUS), P1.B4 (VBUS), P1.B9 (VBUS), Q1.2 (S), R20.1
- new net: D11.1 (K), R23.1
- new net: R6.2, U2.5 (FAULT)
- new net: D10.1 (K), R22.1
- new net: D9.1 (K), R21.1
- new net: D6.1 (K), R15.1
- new net: D12.1 (K), R24.1
- new net: R3.2, R4.1, X1.1 (Tri-State)
- new net: P1.A5 (CC), R18.1
- new net: D13.1 (K), R25.1
- new net: P1.B5 (VCONN), R17.1
- new net: D5.1 (K), R14.1
- new net +5VD: D11.2 (A), D8.2 (A), Q1.3 (D)
- new net 5V_BUS_GOOD_LED: D7.2 (A)
- new net ADC_5V: D3.1 (K), R10.1, R9.2
- new net ADC_BATT: D4.1 (K), R11.2, R12.2, R13.1
- new net BOOT_LED: D5.2 (A)
- new net BUS_POWER_GOOD_LED: D6.2 (A)
- new net PROBLEM_LED: D9.2 (A)
- new net USB_D+: P1.A6 (D+)
- new net USB_D-: P1.A7 (D-)
- no-connect marks 0 -> 1
Other:
- note added: "32768 watch crystal for RTC"
- note added: "5V POWER GOOD LED"
- note added: "5V range measures from 0-2.5V"
- note added: "BOOT LED"
- note added: "BUS POWER GOOD LED"
- note added: "PROBLEM LED"
- note added: "VBUS range from 0 - 2.8V [0V bus to 16.8V bus]"
- moved on the sheet: U1

Commit message: Woo
Parts:
- added C21, C22, C27, C28, C29: 1u, Capacitor_SMD:C_0805_2012Metric, symbol Device:C_Small
- added C23, C24, C25, C26: 100n, Capacitor_SMD:C_0805_2012Metric, symbol Device:C_Small
- added R26, R27: 4k7, Resistor_SMD:R_0805_2012Metric, symbol Device:R_Small_US
- added R28, R29: 10k, Resistor_SMD:R_0805_2012Metric, symbol Device:R_Small_US
- C1, C10, C11, C12, C13, C14, C15, C16, C17, C18, C19, C2, C20, C3, C4, C5, C6, C7, C8, C9: footprint Capacitor_SMD:C_0603_1608Metric -> Capacitor_SMD:C_0805_2012Metric
- D1, D2, D3, D4, D8: footprint (none) -> Diode_SMD:D_SOD-123
- D10, D11, D12, D13, D5, D6, D7, D9: footprint (none) -> LED_SMD:LED_0805_2012Metric
- P1: footprint (none) -> Connector_USB:USB_C_Receptacle_GCT_USB4105-xx-A_16P_TopMnt_Horizontal
- R1, R10, R11, R12, R13, R14, R15, R16, R17, R18, R19, R2, R20, R21, R22, R23, R24, R25, R3, R4, R5, R6, R7, R8, R9: footprint Resistor_SMD:R_0603_1608Metric -> Resistor_SMD:R_0805_2012Metric
Connections:
- net USB_DM is gone; now on net USB_D-: U1.44 (PA11)
- net USB_DP is gone; now on net USB_D+: U1.45 (PA12)
- net +3V3: now also C23.1, C24.1, C25.1, C26.1, C27.1, C28.1, C29.1, R26.1, R27.1
- net 5V_BUS_GOOD_LED: now also U1.35 (PB14)
- net BOOT_LED: now also U1.34 (PB13)
- net BUS_POWER_GOOD_LED: now also U1.36 (PB15)
- net CANH_0: now also J1.B13 (CANH_0); no longer J1.B12 (CANH_0)
- net CANL_0: now also J1.B12 (CANL_0); no longer J1.B13 (CANL_0)
- net ESC_0: now also U1.22 (PA6); no longer U1.27 (PB1)
- net ESC_1: now also U1.23 (PA7); no longer U1.26 (PB0)
- net ESC_2: now also U1.26 (PB0); no longer U1.23 (PA7)
- net ESC_3: now also U1.27 (PB1); no longer U1.22 (PA6)
- net ESC_4: now also U1.14 (PA0); no longer U1.17 (PA3)
- net ESC_5: now also U1.15 (PA1); no longer U1.16 (PA2)
- net ESC_6: now also U1.16 (PA2); no longer U1.15 (PA1)
- net ESC_7: now also U1.17 (PA3); no longer U1.14 (PA0)
- net GND: now also C21.2, C22.2, C23.2, C24.2, C25.2, C26.2, C27.2, C28.2, C29.2
- net PROBLEM_LED: now also U1.33 (PB12)
- net i2C_SCL: now also R26.2
- net i2C_SDA: now also R27.2
- net CAN_FAULT: now reaches R6.2, U2.5 (FAULT)
- net CAN_FAULT: now also U1.56 (PB4)
- net ADC_123_IN12: now reaches U1.10 (PC2)
- net ADC_123_IN13: now reaches U1.11 (PC3)
- net ADC_123_IN10: now reaches U1.8 (PC0)
- net ADC_123_IN10: now also D4.1 (K), C22.1, R29.1
- net ADC_123_IN11: now reaches U1.9 (PC1)
- net ADC_123_IN11: now also D3.1 (K), C21.1, R28.1
- net ADC_5V: no longer names the net of R10.1, R9.2
- net ADC_5V: now also R28.2; no longer D3.1 (K)
- net ADC_BATT: no longer names the net of R11.2, R12.2, R13.1
- net ADC_BATT: now also R29.2; no longer D4.1 (K)
Other:
- moved on the sheet: D3, D4
